Commit message: add new dof

File: src/xeno_urdf/xeno_urdf/urdf/xeno_urdf_description.urdf.xacro (robot description, xacro)
@@ -5,15 +5,15 @@
     <inertial>
       <origin
-        xyz="0.305094473393476 0.297832125522315 0.159681027542379"
-        rpy="0 0 0" />
-      <mass
-        value="8.34373922145942" />
-      <inertia
-        ixx="0.0469906760740281"
-        ixy="5.14839360689645E-05"
-        ixz="6.47739202877026E-07"
-        iyy="0.0564978768313125"
-        iyz="-1.02031036586264E-07"
-        izz="0.0340441540583983" />
+        xyz="0.26669695579372 -0.242025752926975 0.0430843772309064"
+        rpy="0 0 0" />
+      <mass
+        value="2.67946025521633" />
+      <inertia
+        ixx="0.0247505610420922"
+        ixy="1.20986595669565E-08"
+        ixz="3.25666768339599E-05"
+        iyy="0.0352698053676739"
+        iyz="1.26675265404138E-09"
+        izz="0.0311353357370667" />
     </inertial>
     <visual>
@@ -28,5 +28,5 @@
         name="">
         <color
-          rgba="0.898039215686275 0.917647058823529 0.929411764705882 1" />
+          rgba="0.792156862745098 0.819607843137255 0.933333333333333 1" />
       </material>
     </visual>
@@ -45,15 +45,15 @@
     <inertial>
       <origin
-        xyz="-0.203417099023048 0.249999999169318 -0.0147118213931048"
-        rpy="0 0 0" />
-      <mass
-        value="0.665767546458287" />
-      <inertia
-        ixx="6.50274527224072E-05"
-        ixy="-2.74978722993329E-18"
-        ixz="-5.68725101029244E-06"
-        iyy="0.00800853644421888"
-        iyz="2.68466855544117E-19"
-        izz="0.00798296332389548" />
+        xyz="0.185028595714662 -0.00832277412155959 -0.178922873353644"
+        rpy="0 0 0" />
+      <mass
+        value="0.331227493236693" />
+      <inertia
+        ixx="0.00359557900980095"
+        ixy="8.1925548172336E-13"
+        ixz="4.10157129333264E-18"
+        iyy="0.00357618701291859"
+        iyz="6.09931701507021E-18"
+        izz="6.20714942709694E-05" />
     </inertial>
     <visual>
@@ -68,5 +68,5 @@
         name="">
         <color
-          rgba="1 1 1 1" />
+          rgba="0.792156862745098 0.819607843137255 0.933333333333333 1" />
       </material>
     </visual>
@@ -78,204 +78,4 @@
         <mesh
           filename="package://xeno_urdf/xeno_urdf/meshes/link1.STL" />
-      </geometry>
-    </collision>
-  </link>
-  <link
-    name="link_2">
-    <inertial>
-      <origin
-        xyz="0.324490821488572 0.170056267864949 0.028582704465656"
-        rpy="0 0 0" />
-      <mass
-        value="1.21417100402845" />
-      <inertia
-        ixx="0.0065316705527893"
-        ixy="4.70515716369336E-07"
-        ixz="1.97461826682341E-08"
-        iyy="0.0083422227460292"
-        iyz="-4.96570020126472E-08"
-        izz="0.0147593176708924" />
-    </inertial>
-    <visual>
-      <origin
-        xyz="0 0 0"
-        rpy="0 0 0" />
-      <geometry>
-        <mesh
-          filename="package://xeno_urdf/xeno_urdf/meshes/link2.STL" />
-      </geometry>
-      <material
-        name="">
-        <color
-          rgba="0.898039215686275 0.917647058823529 0.929411764705882 1" />
-      </material>
-    </visual>
-    <collision>
-      <origin
-        xyz="0 0 0"
-        rpy="0 0 0" />
-      <geometry>
-        <mesh
-          filename="package://xeno_urdf/xeno_urdf/meshes/link2.STL" />
-      </geometry>
-    </collision>
-  </link>
-  <link
-    name="link_3">
-    <inertial>
-      <origin
-        xyz="-0.0414561721258744 -0.381930292723158 0.0296102021695027"
-        rpy="0 0 0" />
-      <mass
-        value="0.246364304381205" />
-      <inertia
-        ixx="0.000115401552196979"
-        ixy="-1.32414952808114E-05"
-        ixz="4.41732232362797E-09"
-        iyy="3.73447914211717E-05"
-        iyz="5.79263428605455E-08"
-        izz="0.00015058989135556" />
-    </inertial>
-    <visual>
-      <origin
-        xyz="0 0 0"
-        rpy="0 0 0" />
-      <geometry>
-        <mesh
-          filename="package://xeno_urdf/xeno_urdf/meshes/link3.STL" />
-      </geometry>
-      <material
-        name="">
-        <color
-          rgba="0.647058823529412 0.619607843137255 0.588235294117647 1" />
-      </material>
-    </visual>
-    <collision>
-      <origin
-        xyz="0 0 0"
-        rpy="0 0 0" />
-      <geometry>
-        <mesh
-          filename="package://xeno_urdf/xeno_urdf/meshes/link3.STL" />
-      </geometry>
-    </collision>
-  </link>
-  <link
-    name="link_4">
-    <inertial>
-      <origin
-        xyz="0.000118685682633846 -0.0290479332552551 0.0216100676178127"
-        rpy="0 0 0" />
-      <mass
-        value="0.654215847489834" />
-      <inertia
-        ixx="0.000262176142085516"
-        ixy="-9.269799959598E-08"
-        ixz="-2.98072694512485E-08"
-        iyy="0.000284951782416327"
-        iyz="7.65570845300632E-06"
-        izz="0.000290627371493145" />
-    </inertial>
-    <visual>
-      <origin
-        xyz="0 0 0"
-        rpy="0 0 0" />
-      <geometry>
-        <mesh
-          filename="package://xeno_urdf/xeno_urdf/meshes/link4.STL" />
-      </geometry>
-      <material
-        name="">
-        <color
-          rgba="0.898039215686275 0.917647058823529 0.929411764705882 1" />
-      </material>
-    </visual>
-    <collision>
-      <origin
-        xyz="0 0 0"
-        rpy="0 0 0" />
-      <geometry>
-        <mesh
-          filename="package://xeno_urdf/xeno_urdf/meshes/link4.STL" />
-      </geometry>
-    </collision>
-  </link>
-  <link
-    name="link_5">
-    <inertial>
-      <origin
-        xyz="-0.00100717551069329 -0.0735464148845602 0.0133234657824919"
-        rpy="0 0 0" />
-      <mass
-        value="0.108515356455072" />
-      <inertia
-        ixx="9.54767216463274E-05"
-        ixy="4.94143643072523E-07"
-        ixz="1.50000096456065E-08"
-        iyy="3.08967780686823E-05"
-        iyz="-1.56014329844716E-06"
-        izz="9.8648870587829E-05" />
-    </inertial>
-    <visual>
-      <origin
-        xyz="0 0 0"
-        rpy="0 0 0" />
-      <geometry>
-        <mesh
-          filename="package://xeno_urdf/xeno_urdf/meshes/link5.STL" />
-      </geometry>
-      <material
-        name="">
-        <color
-          rgba="0.847058823529412 0.847058823529412 0.847058823529412 1" />
-      </material>
-    </visual>
-    <collision>
-      <origin
-        xyz="0 0 0"
-        rpy="0 0 0" />
-      <geometry>
-        <mesh
-          filename="package://xeno_urdf/xeno_urdf/meshes/link5.STL" />
-      </geometry>
-    </collision>
-  </link>
-  <link
-    name="link_6">
-    <inertial>
-      <origin
-        xyz="2.27595720048157E-15 5.79310904802455E-15 0.0319755100561606"
-        rpy="0 0 0" />
-      <mass
-        value="0.076783081415109" />
-      <inertia
-        ixx="1.60025819642233E-05"
-        ixy="-1.40105408846634E-08"
-        ixz="4.46890691075213E-20"
-        iyy="1.59769774781377E-05"
-        iyz="1.21395301251223E-18"
-        izz="2.2728267321003E-05" />
-    </inertial>
-    <visual>
-      <origin
-        xyz="0 0 0"
-        rpy="0 0 0" />
-      <geometry>
-        <mesh
-          filename="package://xeno_urdf/xeno_urdf/meshes/link6.STL" />
-      </geometry>
-      <material
-        name="">
-        <color
-          rgba="0.898039215686275 0.917647058823529 0.929411764705882 1" />
-      </material>
-    </visual>
-    <collision>
-      <origin
-        xyz="0 0 0"
-        rpy="0 0 0" />
-      <geometry>
-        <mesh
-          filename="package://xeno_urdf/xeno_urdf/meshes/link6.STL" />
       </geometry>
     </collision>
@@ -285,6 +85,6 @@
     type="prismatic">
     <origin
-      xyz="0.077 0.05 0.189"
-      rpy="3.1416 0 -3.1416" />
+      xyz="0.067202 -0.055049 0.04839"
+      rpy="1.5708 0 -1.5708" />
     <parent
       link="base_link" />
@@ -295,14 +95,54 @@
     <limit
       lower="-0.32"
-      upper="0"
+      upper="0.32"
       effort="0"
       velocity="1.5" />
   </joint>
+  <link
+    name="link_2">
+    <inertial>
+      <origin
+        xyz="-0.147952953542361 0.00721513789627723 0.11139952012947"
+        rpy="0 0 0" />
+      <mass
+        value="1.13992890911822" />
+      <inertia
+        ixx="0.0083301452591185"
+        ixy="8.60827876876126E-09"
+        ixz="1.75396040690603E-06"
+        iyy="0.0142979811659756"
+        iyz="-8.55343268612929E-07"
+        izz="0.00606948576919771" />
+    </inertial>
+    <visual>
+      <origin
+        xyz="0 0 0"
+        rpy="0 0 0" />
+      <geometry>
+        <mesh
+          filename="package://xeno_urdf/xeno_urdf/meshes/link2.STL" />
+      </geometry>
+      <material
+        name="">
+        <color
+          rgba="0.792156862745098 0.819607843137255 0.933333333333333 1" />
+      </material>
+    </visual>
+    <collision>
+      <origin
+        xyz="0 0 0"
+        rpy="0 0 0" />
+      <geometry>
+        <mesh
+          filename="package://xeno_urdf/xeno_urdf/meshes/link2.STL" />
+      </geometry>
+    </collision>
+  </link>
   <joint
     name="joint_2"
     type="prismatic">
     <origin
-      xyz="0.002 0.08 0.006"
-      rpy="3.1416 0 3.1416" />
+      xyz="0.034 2.4196E-05 0.019096"
+      rpy="-3.141 0 3.1416" />
     <parent
       link="link_1" />
@@ -310,7 +150,7 @@
       link="link_2" />
     <axis
-      xyz="1 0 0" />
-    <limit
-      lower="0"
+      xyz="0 0 -1" />
+    <limit
+      lower="-0.35"
       upper="0.35"
       effort="0"
@@ -318,10 +158,50 @@
     />
   </joint>
-  <joint
+  <link
+    name="link_3">
+    <inertial>
+      <origin
+        xyz="0.0232065797639486 0.00113688050742744 0.0100412795305758"
+        rpy="0 0 0" />
+      <mass
+        value="0.241891764846693" />
+      <inertia
+        ixx="0.000103123442652323"
+        ixy="-6.54893775078498E-09"
+        ixz="-1.17529230695251E-05"
+        iyy="0.000137114148084955"
+        iyz="-2.85679717502139E-08"
+        izz="3.61873133027448E-05" />
+    </inertial>
+    <visual>
+      <origin
+        xyz="0 0 0"
+        rpy="0 0 0" />
+      <geometry>
+        <mesh
+          filename="package://xeno_urdf/xeno_urdf/meshes/link3.STL" />
+      </geometry>
+      <material
+        name="">
+        <color
+          rgba="0.898039215686275 0.917647058823529 0.929411764705882 1" />
+      </material>
+    </visual>
+    <collision>
+      <origin
+        xyz="0 0 0"
+        rpy="0 0 0" />
+      <geometry>
+        <mesh
+          filename="package://xeno_urdf/xeno_urdf/meshes/link3.STL" />
+      </geometry>
+    </collision>
+  </link>
+    <joint
     name="joint_3"
     type="prismatic">
     <origin
-      xyz="0.4 -0.07 0.02"
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
Commit message: fix revolute intervene

File: src/xeno_urdf/xeno_urdf/urdf/xeno_urdf_description.urdf.xacro (robot description, xacro)
@@ -221,15 +221,15 @@
     <inertial>
       <origin
-        xyz="0.00439378483254166 0.0254526125657555 -0.00291809449607736"
-        rpy="0 0 0" />
-      <mass
-        value="0.447654712261555" />
-      <inertia
-        ixx="0.000168341404535932"
-        ixy="-7.3258760951443E-06"
-        ixz="3.35279679156922E-06"
-        iyy="0.000211045765692015"
-        iyz="5.11467371879199E-06"
-        izz="0.000171730668874568" />
+        xyz="0.0075553 0.025636 -0.0050399"
+        rpy="0 0 0" />
+      <mass
+        value="0.47365" />
+      <inertia
+        ixx="0.00018548"
+        ixy="-7.0956E-06"
+        ixz="-1.8556E-06"
+        iyy="0.00022296"
+        iyz="4.9602E-06"
+        izz="0.00018459" />
     </inertial>
     <visual>
@@ -244,5 +244,5 @@
         name="">
         <color
-          rgba="0.250980392156863 0.250980392156863 0.250980392156863 1" />
+          rgba="0.25098 0.25098 0.25098 1" />
       </material>
     </visual>
@@ -280,15 +280,15 @@
     <inertial>
       <origin
-        xyz="0.00108717237907943 0.023015795700147 7.26331907813238E-10"
-        rpy="0 0 0" />
-      <mass
-        value="0.299443586631998" />
-      <inertia
-        ixx="0.000105388224794985"
-        ixy="5.77780829764042E-07"
-        ixz="2.4259790039032E-09"
-        iyy="0.000130873026168991"
-        iyz="2.71050543121376E-20"
-        izz="0.000103481334324279" />
+        xyz="-0.0022472 0.028349 1.3904E-10"
+        rpy="0 0 0" />
+      <mass
+        value="0.32655" />
+      <inertia
+        ixx="0.00013266"
+        ixy="4.6197E-06"
+        ixz="2.426E-09"
+        iyy="0.00013588"
+        iyz="7.8715E-14"
+        izz="0.0001222" />
     </inertial>
     <visual>
@@ -339,15 +339,15 @@
     <inertial>
       <origin
-        xyz="-0.00901165823398339 0.0201192726579273 0.0097262995405353"
-        rpy="0 0 0" />
-      <mass
-        value="0.569307015021012" />
-      <inertia
-        ixx="0.00021937666575888"
-        ixy="-2.75634795597272E-06"
-        ixz="1.94289786271747E-05"
-        iyy="0.000295160570942927"
-        iyz="3.0744613027115E-06"
-        izz="0.000220002969096714" />
+        xyz="-0.011521 0.021899 0.012318"
+        rpy="0 0 0" />
+      <mass
+        value="0.51621" />
+      <inertia
+        ixx="0.00019251"
+        ixy="2.8892E-07"
+        ixz="1.8201E-05"
+        iyy="0.00025598"
+        iyz="1.1486E-08"
+        izz="0.00019315" />
     </inertial>
     <visual>
@@ -398,15 +398,15 @@
     <inertial>
       <origin
-        xyz="-0.00884716965172472 5.8063530095076E-09 7.9260683849558E-09"
-        rpy="0 0 0" />
-      <mass
-        value="0.0441931131241815" />
-      <inertia
-        ixx="1.86781683229588E-05"
-        ixy="-3.22043202251819E-12"
-        ixz="-3.36854010207685E-12"
-        iyy="1.15856573921313E-05"
-        iyz="-7.70011464899261E-12"
-        izz="1.15856654956983E-05" />
+        xyz="-0.0088472 4.0935E-09 1.119E-08"
+        rpy="0 0 0" />
+      <mass
+        value="0.044193" />
+      <inertia
+        ixx="1.8678E-05"
+        ixy="-3.2204E-12"
+        ixz="-3.3685E-12"
+        iyy="1.1586E-05"
+        iyz="-7.7001E-12"
+        izz="1.1586E-05" />
     </inertial>
     <visual>

Commit message: add limit

File: src/xeno_urdf/xeno_urdf/urdf/xeno_urdf_description.urdf.xacro (robot description, xacro)
@@ -93,7 +93,8 @@
     <axis
       xyz="0 1 0" />
-    <limit
-      lower="-0.32"
-      upper="0.32"
+    <!-- 298.37mm -->
+    <limit
+      lower="0"
+      upper="0.29"
       effort="0"
       velocity="1.5" />
@@ -139,4 +140,5 @@
     </collision>
   </link>
+  <!-- 298.37mm -->
   <joint
     name="joint_2"
@@ -152,5 +154,5 @@
       xyz="0 0 -1" />
     <limit
-      lower="-0.35"
+      lower="0"
       upper="0.35"
       effort="0"
@@ -198,4 +200,5 @@
     </collision>
   </link>
+    <!-- 380mm -->
     <joint
     name="joint_3"
@@ -209,8 +212,8 @@
       link="link_3" />
     <axis
-      xyz="0 0 -1" />
-    <limit
-      lower="-0.38"
-      upper="0.38"
+      xyz="0 0 1" />
+    <limit
+      lower="0"
+      upper="0.17"
       effort="0"
       velocity="1.5"
